File: plankSplit_right.kicad_pcb (KiCad board)
At the start: 2 copper layers, 122.2 x 127.3 mm, 105 parts, among them P1 USB_A, SW0:1 SPACE, SW0:2 ENTER, SW0:3 ALTGR, SW0:4 FN_R, SW0:5 MOD4, SW0:6 CTRL_R, SW1:1 B, SW1:2 M, SW1:3 ,, SW1:4 ., SW1:5 J, SW1:6 END, SW2:1 S, SW2:2 N, SW2:3 R, SW2:4 T, SW2:5 D, SW2:6 Y, SW3:1 K, SW3:2 H, SW3:3 G, SW3:4 F, SW3:5 Q, SW3:6 ẞ, SW4:1 6, SW4:2 7, SW4:3 8, SW4:4 9, SW4:5 0, SW4:6 BCKSPC, U1 ATmega32U4-AU, X1 CRYSTAL

Commit message: Rev1.0
Parts:
- removed 100nF1: CBUS, Capacitors_SMD:C_0402
- removed 10k1: R, Resistors_SMD:R_0805
- removed the REF** at (102.1, 34.2)
- removed the REF** at (117.3, 95.2)
- removed the REF** at (117.3, 56.4)
- removed the REF** at (23.7, 134.7)
- removed the REF** at (135.0, 134.9)
- removed the REF** at (79.5, 94.2)
- removed the REF** at (136.7, 33.8)
- removed the REF** at (72.1, 32.0)
- removed the REF** at (61.5, 22.1)
- removed the REF** at (68.1, 26.7)
- removed the REF** at (105.9, 17.8)
- removed the REF** at (22.6, 16.5)
- removed the REF** at (30.2, 20.8)
- removed the REF** at (41.4, 133.6)
- removed the REF** at (79.0, 115.1)
- removed the REF** at (42.4, 96.0)
- removed the REF** at (41.9, 56.4)
- removed the REF** at (78.0, 56.1)
- removed the REF** at (117.3, 132.1)
- removed RJ11: CONN_6, mmmm:rj11
- removed SW_PRGRM1: PRGRM, Buttons_Switches_SMD:SW_SPST_SKQG
- added C8: 1uF, Capacitors_SMD:C_0603, F.Cu at (53.4, 26.7)
- added CBUS1: 100nF, Capacitors_SMD:C_0603, F.Cu at (45.0, 15.3)
- added R1: 10k, Resistors_SMD:R_0603, F.Cu at (108.0, 31.4)
- added REF**: VIA_06MM, mmmm:VIA_06MM, F.Cu at (40.1, 15.2)
- added REF**: VIA_06MM, mmmm:VIA_06MM, F.Cu at (79.5, 95.5)
- added REF**: VIA_06MM, mmmm:VIA_06MM, F.Cu at (117.6, 95.0)
- added REF**: VIA_06MM, mmmm:VIA_06MM, F.Cu at (63.0, 21.6)
- added REF**: VIA_06MM, mmmm:VIA_06MM, F.Cu at (51.6, 30.5)
- added REF**: VIA_06MM, mmmm:VIA_06MM, F.Cu at (71.4, 32.0)
- added REF**: VIA_06MM, mmmm:VIA_06MM, F.Cu at (117.6, 57.1)
- added REF**: VIA_06MM, mmmm:VIA_06MM, F.Cu at (42.9, 95.8)
- added REF**: VIA_06MM, mmmm:VIA_06MM, F.Cu at (29.0, 21.1)
- added REF**: VIA_06MM, mmmm:VIA_06MM, F.Cu at (102.4, 20.6)
- added REF**: VIA_06MM, mmmm:VIA_06MM, F.Cu at (102.1, 33.6)
- added REF**: VIA_06MM, mmmm:VIA_06MM, F.Cu at (68.3, 26.7)
- added REF**: VIA_06MM, mmmm:VIA_06MM, F.Cu at (102.4, 18.0)
- added REF**: VIA_06MM, mmmm:VIA_06MM, F.Cu at (130.3, 31.0)
- added REF**: 1pin, Connect:1pin, F.Cu at (136.7, 16.8)
- added REF**: 1pin, Connect:1pin, F.Cu at (79.5, 75.7)
- added REF**: 1pin, Connect:1pin, F.Cu at (23.1, 135.4)
- added REF**: 1pin, Connect:1pin, F.Cu at (136.7, 135.4)
- added REF**: 1pin, Connect:1pin, F.Cu at (23.1, 16.8)
- added REF**: VIA_06MM, mmmm:VIA_06MM, F.Cu at (42.2, 56.1)
- added REF**: VIA_06MM, mmmm:VIA_06MM, F.Cu at (79.2, 31.5)
- added REF**: VIA_06MM, mmmm:VIA_06MM, F.Cu at (78.0, 56.1)
- added SW_RST1: SWRST, Buttons_Switches_SMD:SW_SPST_SKQG, F.Cu at (117.1, 30.2)
- added USBCONN1: CONN_5, mmmm:usb-b-mini-female, F.Cu at (124.5, 12.4)
- added USBCONN2: CONN_5, mmmm:usb-b-mini-female, B.Cu at (124.5, 12.4)
- C1, C2: value C -> 22pF; footprint Capacitors_SMD:C_0402 -> Capacitors_SMD:C_0603
- C3, C4, C5, C6, C7: value C -> 100nF; footprint Capacitors_SMD:C_0805 -> Capacitors_SMD:C_0603
- D34: footprint Diodes_SMD:MiniMELF_Standard -> Diodes_SMD:SMA_Standard
- R_LED1, R_LED2, R_LED3: footprint Resistors_SMD:R_0402 -> Resistors_SMD:R_0603
- USB_DM_R1, USB_DP_R1, VCCCHECK1: footprint Resistors_SMD:R_0805 -> Resistors_SMD:R_0603
- moved C5 0.25 mm to (47.8, 16.3)
- moved C4 0.24 mm to (43.4, 24.1)
- moved C6 0.18 mm to (43.4, 33.1)
Connections:
- U1 pad 6: (no net) -> /UCAP
- U1 pad 8: /SS -> (no net)
Routing:
- net /SS: track 74.6 -> 0.00 mm
- net /SCLK: track 73.3 -> 102.9 mm, vias 0 -> 1
- net /DATA2: track 73.9 -> 97.6 mm, vias 0 -> 1
- net /DATA1: track 76.5 -> 97.4 mm, vias 0 -> 1
- net /P14_VCC: track 301.1 -> 316.3 mm, vias 10 -> 11
- net /VBus: track 11.5 -> 22.3 mm, vias 2 -> 4
- net /UGND: track 63.2 -> 70.6 mm, vias 9 -> 8
- net /UCAP: track 0.00 -> 4.40 mm, vias 0 -> 1
- net (no net): track 0.00 -> 2.87 mm, vias 1 -> 0
- net /RST: track 222.3 -> 221.5 mm
- net Net-(D32-Pad1): track 2.04 -> 2.80 mm
- net Net-(D31-Pad1): track 2.04 -> 2.80 mm
- net Net-(D33-Pad1): track 2.04 -> 2.80 mm
